File: hw/schematic/kiosk_power_revB.brd (EAGLE design)
At the start: 35.7 x 46 mm, 26 parts, among them J1 POWER_JACK, K1 BT-5-S, T1 BC547, T2 BC517, T3 IRLU7843TO251AA

Commit message: hw: schematic: Updated schematic
Increased relay coil series resistance to 220 ohms,
which decreases power consumption.

Signed-off-by: Jan Siegmund <jsiegmun@hm.edu>
Parts:
- R8: value 120 -> 220
Changed lines of the file:
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@@
 <element name="R7" library="resistor" library_urn="urn:adsk.eagle:library:348" package="0207/7" package3d_urn="urn:adsk.eagle:package:25942/1" value="10k" x="81.5975" y="0.15875" rot="R180"/>
 <element name="C4" library="resistor" library_urn="urn:adsk.eagle:library:348" package="E2-5" package3d_urn="urn:adsk.eagle:package:25833/1" value="470u" x="83.97875" y="23.1775" rot="R180"/>
-<element name="R8" library="resistor" library_urn="urn:adsk.eagle:library:348" package="0207/7" package3d_urn="urn:adsk.eagle:package:25942/1" value="120" x="76.04125" y="24.28875" rot="R270"/>
+<element name="R8" library="resistor" library_urn="urn:adsk.eagle:library:348" package="0207/7" package3d_urn="urn:adsk.eagle:package:25942/1" value="220" x="76.04125" y="24.28875" rot="R270"/>
 <element name="PI3_FEEDBACK" library="kiosk" package="1X01/90" value="" x="86.995" y="2.06375" rot="R270"/>
 </elements>
